Commit message: Added robot world

File: urdf/ddrobot/robot.urdf (robot description, URDF)
Before this commit: robot ddrobot, 4 links, 3 joints
Links:
- link chasis: mass 5 -> 0.1; geometry collision cylinder length=0.15 radius=0.05; collision cylinder length=0.15 radius=0.4
- link left_wheel: mass 0.5 -> 0.015
- link right_wheel: mass 0.5 -> 0.015

File: urdf/ddrobot/xacro/chasis.xacro (robot description, xacro)
@@ -17,10 +17,10 @@
         <link name="chasis">
             <!-- Main Robot Body -->
-            <visual name="main_chasis">
+            <visual>
                 <origin xyz="0.0 0.0 0.0" rpy="0.0 0.0 0.0" />
                 <geometry>
                     <cylinder radius="${chasis_radius}" length="${chasis_height}"/>
                 </geometry>
-                <material name="yellow" />
+                <material name="red" />
             </visual>
             <collision>
@@ -35,10 +35,10 @@
             </inertial>
             <!-- Passive Wheel Holder -->
-            <visual name="passive_wheel_holder">
+            <visual>
                 <origin xyz="0.2 0 -0.075" rpy="0 0 0" />
                 <geometry>
                     <cylinder radius="${passive_wheel_holder_radius}" length="${passive_wheel_holder_height}"/>
                 </geometry>
-                <material name="yellow" />
+                <material name="red" />
             </visual>
             <collision>
@@ -53,10 +53,10 @@
             </inertial>
             <!-- Passive Wheel -->
-            <visual name="passive_wheel">
+            <visual>
                 <origin xyz="0.2 0 -0.15" rpy="0 0 0" />
                 <geometry>
                     <sphere radius="${passive_wheel_radius}" />
                 </geometry>
-                <material name="yellow" />
+                <material name="red" />
             </visual>
             <collision>

File: urdf/ddrobot/xacro/gazebo.xacro (robot description, xacro)
@@ -2,5 +2,5 @@
 <robot xmlns:xacro="http://www.ros.org/wiki/xacro">
     <gazebo reference="chasis">
-        <material>Gazebo/Yellow</material>
+        <material>Gazebo/Red</material>
     </gazebo>
     <gazebo reference="right_wheel">

File: urdf/ddrobot/xacro/materials.xacro (robot description, xacro)
@@ -4,6 +4,6 @@
         <color rgba="0 0 0 1"/>
     </material>
-    <material name="yellow">
-        <color rgba="1 1 0 1"/>
+    <material name="red">
+        <color rgba="1 0 0 1"/>
     </material>
 </robot>

Commit message: can spawn multiple robots with description into gazebo, rviz off for now

File: urdf/ddrobot/robot.urdf (robot description, URDF)
Before this commit: robot ddrobot, 4 links, 3 joints
Links:
- link chasis: geometry collision cylinder length=0.018 radius=0.01; collision cylinder length=0.025 radius=0.0825
- link left_wheel: geometry collision cylinder length=0.008 radius=0.035; visual cylinder length=0.008 radius=0.035
- link right_wheel: geometry collision cylinder length=0.008 radius=0.035; visual cylinder length=0.008 radius=0.035

File: urdf/ddrobot/robot.xacro (robot description, xacro)
@@ -10,5 +10,7 @@
     <xacro:chasis />
     <!-- Robot Wheels -->
-    <xacro:wheel prefix="left" offset="0.45" />
-    <xacro:wheel prefix="right" offset="-0.45" />
+    <xacro:wheel prefix="right" suffix="front" offset_x="${chasis_length/2 - 0.1}" offset_y="${chasis_width/2 + 0.05}" />
+    <xacro:wheel prefix="left" suffix="front" offset_x="${chasis_length/2 - 0.1}" offset_y="${-(chasis_width/2 + 0.05)}" />
+    <xacro:wheel prefix="right" suffix="back" offset_x="${-(chasis_length/2 - 0.1)}" offset_y="${chasis_width/2 + 0.05}" />
+    <xacro:wheel prefix="left" suffix="back" offset_x="${-(chasis_length/2 - 0.1)}" offset_y="${-(chasis_width/2 + 0.05)}" />
 </robot>

File: urdf/ddrobot/xacro/chasis.xacro (robot description, xacro)
@@ -1,24 +1,39 @@
 <?xml version="1.0"?>
 <robot xmlns:xacro="http://www.ros.org/wiki/xacro">
+    <xacro:property name="head_mass" value="0.2" />
+    <xacro:property name="head_radius" value="0.15" />
+    <xacro:property name="head_inertia_calc" value="${(2/5) * head_mass * (head_radius * head_radius)}" />
     <xacro:property name="chasis_mass" value="0.1" />
-    <xacro:property name="chasis_radius" value="0.4" />
-    <xacro:property name="chasis_height" value="0.15" />
-    <xacro:property name="chasis_inertia_calc" value="${(1/12) * chasis_mass * ((3 * (chasis_radius * chasis_radius)) + (chasis_height * chasis_height))}" />
-    <xacro:property name="chasis_inertia_calc_izz" value="${(1/2) * chasis_mass * (chasis_radius * chasis_radius)}" />
-    <xacro:property name="passive_wheel_holder_mass" value="0.02" />
-    <xacro:property name="passive_wheel_holder_radius" value="0.05" />
-    <xacro:property name="passive_wheel_holder_height" value="0.15" />
-    <xacro:property name="passive_wheel_holder_inertia_calc" value="${(1/12) * passive_wheel_holder_mass * ((3 * (passive_wheel_holder_radius * chasis_radius)) + (passive_wheel_holder_height * passive_wheel_holder_height))}" />
-    <xacro:property name="passive_wheel_holder_inertia_calc_izz" value="${(1/2) * passive_wheel_holder_mass * (passive_wheel_holder_radius * chasis_radius)}" />
-    <xacro:property name="passive_wheel_mass" value="0.02" />
-    <xacro:property name="passive_wheel_radius" value="0.05" />
-    <xacro:property name="passive_wheel_inertia_calc" value="${(2/5) * passive_wheel_mass * (passive_wheel_radius * passive_wheel_radius)}" />
+    <xacro:property name="chasis_width" value="0.8" />
+    <xacro:property name="chasis_height" value="0.25" />
+    <xacro:property name="chasis_length" value="1" />
+    <xacro:property name="chasis_inertia_calc_ixx" value="${(1/12) * chasis_mass * ((chasis_height * chasis_height) + (chasis_length * chasis_length))}" />
+    <xacro:property name="chasis_inertia_calc_iyy" value="${(1/12) * chasis_mass * ((chasis_width * chasis_width) + (chasis_height * chasis_height))}" />
+    <xacro:property name="chasis_inertia_calc_izz" value="${(1/12) * chasis_mass * ((chasis_width * chasis_width) + (chasis_length * chasis_length))}" />
     <xacro:macro name="chasis">
         <link name="chasis">
+            <!-- Robot Head -->
+            <visual>
+                <origin xyz="0.3 0 0.25" rpy="0.0 0.0 0.0" />
+                <geometry>
+                    <sphere radius="${head_radius}" />
+                </geometry>
+                <material name="red" />
+            </visual>
+            <collision>
+                <origin xyz="0.3 0 0.25" rpy="0.0 0.0 0.0" />
+                <geometry>
+                    <sphere radius="${head_radius}" />
+                </geometry>
+            </collision>
+            <inertial>
+                <mass value="${chasis_mass}"/>
+                <inertia ixx="${head_inertia_calc}" ixy="0.0" ixz="0.0" iyy="${head_inertia_calc}" iyz="0.0" izz="${head_inertia_calc}"/>
+            </inertial>
             <!-- Main Robot Body -->
             <visual>
                 <origin xyz="0.0 0.0 0.0" rpy="0.0 0.0 0.0" />
                 <geometry>
-                    <cylinder radius="${chasis_radius}" length="${chasis_height}"/>
+                    <box size="${chasis_length} ${chasis_width} ${chasis_height}" />
                 </geometry>
                 <material name="red" />
@@ -27,46 +42,10 @@
                 <origin xyz="0.0 0.0 0.0" rpy="0.0 0.0 0.0" />
                 <geometry>
-                    <cylinder radius="${chasis_radius}" length="${chasis_height}"/>
+                    <box size="${chasis_length} ${chasis_width} ${chasis_height}" />
                 </geometry>
             </collision>
             <inertial>
                 <mass value="${chasis_mass}"/>
-                <inertia ixx="${chasis_inertia_calc}" ixy="0.0" ixz="0.0" iyy="${chasis_inertia_calc}" iyz="0.0" izz="${chasis_inertia_calc_izz}"/>
-            </inertial>
-            <!-- Passive Wheel Holder -->
-            <visual>
-                <origin xyz="0.2 0 -0.075" rpy="0 0 0" />
-                <geometry>
-                    <cylinder radius="${passive_wheel_holder_radius}" length="${passive_wheel_holder_height}"/>
-                </geometry>
-                <material name="red" />
-            </visual>
-            <collision>
-                <origin xyz="0.2 0 -0.075" rpy="0 0 0" />
-                <geometry>
-                    <cylinder radius="${passive_wheel_holder_radius}" length="${passive_wheel_holder_height}"/>
-                </geometry>
-            </collision>
-            <inertial>
-                <mass value="${passive_wheel_holder_mass}"/>
-                <inertia ixx="${passive_wheel_holder_inertia_calc}" ixy="0.0" ixz="0.0" iyy="${passive_wheel_holder_inertia_calc}" iyz="0.0" izz="${passive_wheel_holder_inertia_calc}"/>
-            </inertial>
-            <!-- Passive Wheel -->
-            <visual>
-                <origin xyz="0.2 0 -0.15" rpy="0 0 0" />
-                <geometry>
-                    <sphere radius="${passive_wheel_radius}" />
-                </geometry>
-                <material name="red" />
-            </visual>
-            <collision>
-                <origin xyz="0.2 0 -0.15" rpy="0 0 0" />
-                <geometry>
-                    <sphere radius="${passive_wheel_radius}" />
-                </geometry>
-            </collision>
-            <inertial>
-                <mass value="${passive_wheel_mass}"/>
-                <inertia ixx="${passive_wheel_inertia_calc}" ixy="0.0" ixz="0.0" iyy="${passive_wheel_inertia_calc}" iyz="0.0" izz="${passive_wheel_inertia_calc}"/>
+                <inertia ixx="${chasis_inertia_calc_ixx}" ixy="0.0" ixz="0.0" iyy="${chasis_inertia_calc_iyy}" iyz="0.0" izz="${chasis_inertia_calc_izz}"/>
             </inertial>
         </link>

File: urdf/ddrobot/xacro/gazebo.xacro (robot description, xacro)
@@ -4,8 +4,14 @@
         <material>Gazebo/Red</material>
     </gazebo>
-    <gazebo reference="right_wheel">
+    <gazebo reference="right_front_wheel">
         <material>Gazebo/Black</material>
     </gazebo>
-    <gazebo reference="left_wheel">
+    <gazebo reference="right_back_wheel">
+        <material>Gazebo/Black</material>
+    </gazebo>
+    <gazebo reference="left_front_wheel">
+        <material>Gazebo/Black</material>
+    </gazebo>
+    <gazebo reference="left_back_wheel">
         <material>Gazebo/Black</material>
     </gazebo>

File: urdf/studentbot/xacro/wheels.xacro (robot description, xacro)
@@ -6,8 +6,8 @@
     <xacro:property name="wheel_inertia_calc" value="${(1/12) * wheel_mass * ((3 * (wheel_radius * wheel_radius)) + (wheel_height * wheel_height))}" />
     <xacro:property name="wheel_inertia_calc_izz" value="${(1/2) * wheel_mass * (wheel_radius * wheel_radius)}" />
-    <xacro:macro name="wheel" params="prefix suffix offset_x offset_y">
-        <link name="${prefix}_${suffix}_wheel">
+    <xacro:macro name="wheel" params="prefix offset">
+        <link name="${prefix}_wheel">
             <visual>
-                <origin xyz="0 0 0" rpy="${pi/2} 0 0"/>
+                <origin xyz="0.0 0.0 0.0" rpy="${pi/2} 0.0 0.0"/>
                 <geometry>
                     <cylinder radius="${wheel_radius}" length="${wheel_height}"/>
@@ -16,5 +16,5 @@
             </visual>
             <collision>
-                <origin xyz="0 0 0" rpy="${pi/2} 0 0"/>
+                <origin xyz="0.0 0.0 0.0" rpy="${pi/2} 0.0 0.0"/>
                 <geometry>
                     <cylinder radius="${wheel_radius}" length="${wheel_height}"/>
@@ -26,8 +26,8 @@
             </inertial>
         </link>
-        <joint name="joint_${prefix}_${suffix}_wheel" type="continuous">
+        <joint name="joint_${prefix}_wheel" type="continuous">
             <parent link="chasis"/>
-            <child link="${prefix}_${suffix}_wheel"/>
-            <origin xyz="${offset_x} ${offset_y} 0.0" rpy="0.0 0.0 0.0"/>
+            <child link="${prefix}_wheel"/>
+            <origin xyz="0.0 ${offset} 0.0" rpy="0.0 0.0 0.0"/>
             <axis xyz="0.0 1 0.0"/>
         </joint>

Commit message: Added diff_drive controller for wheel joints

File: urdf/ddrobot/robot.urdf (robot description, URDF)
Before this commit: robot ddrobot, 4 links, 3 joints
Links:
- removed link left_wheel
- removed link right_wheel
- added link left_back_wheel, mass 0.015; collision cylinder length=0.1 radius=0.2; visual cylinder length=0.1 radius=0.2
- added link left_front_wheel, mass 0.015; collision cylinder length=0.1 radius=0.2; visual cylinder length=0.1 radius=0.2
- added link right_back_wheel, mass 0.015; collision cylinder length=0.1 radius=0.2; visual cylinder length=0.1 radius=0.2
- added link right_front_wheel, mass 0.015; collision cylinder length=0.1 radius=0.2; visual cylinder length=0.1 radius=0.2
- link chasis: geometry collision box size=1 0.8 0.25; collision sphere radius=0.15
Joints:
- removed joint joint_left_wheel
- removed joint joint_right_wheel
- added joint joint_left_back_wheel: type continuous, parent chasis, child left_back_wheel, origin xyz=-0.4 -0.45 0.0 rpy=0.0 0.0 0.0, axis 0.0 1 0.0
- added joint joint_left_front_wheel: type continuous, parent chasis, child left_front_wheel, origin xyz=0.4 -0.45 0.0 rpy=0.0 0.0 0.0, axis 0.0 1 0.0
- added joint joint_right_back_wheel: type continuous, parent chasis, child right_back_wheel, origin xyz=-0.4 0.45 0.0 rpy=0.0 0.0 0.0, axis 0.0 1 0.0
- added joint joint_right_front_wheel: type continuous, parent chasis, child right_front_wheel, origin xyz=0.4 0.45 0.0 rpy=0.0 0.0 0.0, axis 0.0 1 0.0

File: urdf/ddrobot/robot.xacro (robot description, xacro)
@@ -10,7 +10,7 @@
     <xacro:chasis />
     <!-- Robot Wheels -->
-    <xacro:wheel prefix="right" suffix="front" offset_x="${chasis_length/2 - 0.1}" offset_y="${chasis_width/2 + 0.05}" />
-    <xacro:wheel prefix="left" suffix="front" offset_x="${chasis_length/2 - 0.1}" offset_y="${-(chasis_width/2 + 0.05)}" />
-    <xacro:wheel prefix="right" suffix="back" offset_x="${-(chasis_length/2 - 0.1)}" offset_y="${chasis_width/2 + 0.05}" />
-    <xacro:wheel prefix="left" suffix="back" offset_x="${-(chasis_length/2 - 0.1)}" offset_y="${-(chasis_width/2 + 0.05)}" />
+    <xacro:wheel side="right" position="front" offset_x="${chasis_length/2 - 0.1}" offset_y="${chasis_width/2 + 0.05}" />
+    <xacro:wheel side="left" position="front" offset_x="${chasis_length/2 - 0.1}" offset_y="${-(chasis_width/2 + 0.05)}" />
+    <xacro:wheel side="right" position="back" offset_x="${-(chasis_length/2 - 0.1)}" offset_y="${chasis_width/2 + 0.05}" />
+    <xacro:wheel side="left" position="back" offset_x="${-(chasis_length/2 - 0.1)}" offset_y="${-(chasis_width/2 + 0.05)}" />
 </robot>

File: urdf/ddrobot/xacro/gazebo.xacro (robot description, xacro)
@@ -1,18 +1,33 @@
 <?xml version="1.0"?>
 <robot xmlns:xacro="http://www.ros.org/wiki/xacro">
+    <xacro:macro name="robot_dynamics">
+        <mu1 value="200.0"/>
+        <mu2 value="100.0"/>
+        <kp value="10000000.0" />
+        <kd value="1.0" />
+    </xacro:macro>
+    <!-- Reference to robot links -->
     <gazebo reference="chasis">
         <material>Gazebo/Red</material>
     </gazebo>
     <gazebo reference="right_front_wheel">
+        <xacro:robot_dynamics />
         <material>Gazebo/Black</material>
     </gazebo>
     <gazebo reference="right_back_wheel">
+        <xacro:robot_dynamics />
         <material>Gazebo/Black</material>
     </gazebo>
     <gazebo reference="left_front_wheel">
+        <xacro:robot_dynamics />
         <material>Gazebo/Black</material>
     </gazebo>
     <gazebo reference="left_back_wheel">
+        <xacro:robot_dynamics />
         <material>Gazebo/Black</material>
     </gazebo>
+    <!-- Gazebo Plugins -->
+    <gazebo>
+        <plugin name="gazebo_ros_control" filename="libgazebo_ros_control.so"></plugin>
+    </gazebo>
 </robot>

File: urdf/ddrobot/xacro/wheels.xacro (robot description, xacro)
@@ -1,4 +1,5 @@
 <?xml version="1.0"?>
 <robot xmlns:xacro="http://www.ros.org/wiki/xacro">
+    <xacro:include filename="$(find machine_vision_bonus)/urdf/ddrobot/xacro/transmissions.xacro"/>
     <xacro:property name="wheel_mass" value="0.015" />
     <xacro:property name="wheel_radius" value="0.2" />
@@ -6,6 +7,6 @@
     <xacro:property name="wheel_inertia_calc" value="${(1/12) * wheel_mass * ((3 * (wheel_radius * wheel_radius)) + (wheel_height * wheel_height))}" />
     <xacro:property name="wheel_inertia_calc_izz" value="${(1/2) * wheel_mass * (wheel_radius * wheel_radius)}" />
-    <xacro:macro name="wheel" params="prefix suffix offset_x offset_y">
-        <link name="${prefix}_${suffix}_wheel">
+    <xacro:macro name="wheel" params="side position offset_x offset_y">
+        <link name="${side}_${position}_wheel">
             <visual>
                 <origin xyz="0 0 0" rpy="${pi/2} 0 0"/>
@@ -26,10 +27,12 @@
             </inertial>
         </link>
-        <joint name="joint_${prefix}_${suffix}_wheel" type="continuous">
+        <joint name="joint_${side}_${position}_wheel" type="continuous">
             <parent link="chasis"/>
-            <child link="${prefix}_${suffix}_wheel"/>
+            <child link="${side}_${position}_wheel"/>
             <origin xyz="${offset_x} ${offset_y} 0.0" rpy="0.0 0.0 0.0"/>
             <axis xyz="0.0 1 0.0"/>
         </joint>
+        <!-- Robot Joints' Transmission -->
+        <xacro:wheel_transmission wheelJointName="joint_${side}_${position}_wheel"  />
     </xacro:macro>
 </robot>
