Commit message: scene set correctly

File: urdf/ddrobot/robot.xacro (robot description, xacro)
@@ -3,6 +3,6 @@
     <xacro:include filename="$(find machine_vision_bonus)/urdf/ddrobot/xacro/chasis.xacro"/>
     <xacro:include filename="$(find machine_vision_bonus)/urdf/ddrobot/xacro/wheels.xacro"/>
+    <xacro:include filename="$(find machine_vision_bonus)/urdf/ddrobot/xacro/gazebo.xacro"/>
     <xacro:include filename="$(find machine_vision_bonus)/urdf/ddrobot/xacro/materials.xacro"/>
-    <xacro:include filename="$(find machine_vision_bonus)/urdf/ddrobot/xacro/gazebo.xacro"/>
     <!-- Robot Base Footprint -->
     <link name="base_footprint"></link>
@@ -10,7 +10,7 @@
     <xacro:chasis />
     <!-- Robot Wheels -->
-    <xacro:wheel side="right" position="front" offset_x="${chasis_length/2 - 0.1}" offset_y="${chasis_width/2 + 0.05}" />
-    <xacro:wheel side="left" position="front" offset_x="${chasis_length/2 - 0.1}" offset_y="${-(chasis_width/2 + 0.05)}" />
-    <xacro:wheel side="right" position="back" offset_x="${-(chasis_length/2 - 0.1)}" offset_y="${chasis_width/2 + 0.05}" />
-    <xacro:wheel side="left" position="back" offset_x="${-(chasis_length/2 - 0.1)}" offset_y="${-(chasis_width/2 + 0.05)}" />
+    <xacro:wheel side="right" position="front" offset_x="${chasis_length/2 - 0.1}" offset_y="${-(chasis_width/2 + 0.05)}" />
+    <xacro:wheel side="left" position="front" offset_x="${chasis_length/2 - 0.1}" offset_y="${chasis_width/2 + 0.05}" />
+    <xacro:wheel side="right" position="back" offset_x="${-(chasis_length/2 - 0.1)}" offset_y="${-(chasis_width/2 + 0.05)}" />
+    <xacro:wheel side="left" position="back" offset_x="${-(chasis_length/2 - 0.1)}" offset_y="${chasis_width/2 + 0.05}" />
 </robot>

File: urdf/ddrobot/xacro/chasis.xacro (robot description, xacro)
@@ -12,8 +12,8 @@
     <xacro:property name="chasis_inertia_calc_izz" value="${(1/12) * chasis_mass * ((chasis_width * chasis_width) + (chasis_length * chasis_length))}" />
     <xacro:macro name="chasis">
-        <link name="chasis">
-            <!-- Robot Head -->
+        <!-- Robot Head Mount -->
+        <link name="head_mount">
             <visual>
-                <origin xyz="0.3 0 0.25" rpy="0.0 0.0 0.0" />
+                <origin xyz="0 0 0" rpy="0.0 0.0 0.0" />
                 <geometry>
                     <sphere radius="${head_radius}" />
@@ -22,5 +22,5 @@
             </visual>
             <collision>
-                <origin xyz="0.3 0 0.25" rpy="0.0 0.0 0.0" />
+                <origin xyz="0 0 0" rpy="0.0 0.0 0.0" />
                 <geometry>
                     <sphere radius="${head_radius}" />
@@ -31,5 +31,12 @@
                 <inertia ixx="${head_inertia_calc}" ixy="0.0" ixz="0.0" iyy="${head_inertia_calc}" iyz="0.0" izz="${head_inertia_calc}"/>
             </inertial>
-            <!-- Main Robot Body -->
+        </link>
+        <joint name="joint_chasis__head_mount" type="fixed">
+            <origin xyz="0.35 0 0.23" rpy="0.0 0.0 0.0" />
+            <parent link="chasis"/>
+            <child link="head_mount"/>
+        </joint>
+        <!-- Main Robot Body  -->
+        <link name="chasis">
             <visual>
                 <origin xyz="0.0 0.0 0.0" rpy="0.0 0.0 0.0" />

File: urdf/ddrobot/xacro/gazebo.xacro (robot description, xacro)
@@ -9,4 +9,7 @@
     <!-- Reference to robot links -->
     <gazebo reference="chasis">
+        <material>Gazebo/Red</material>
+    </gazebo>
+    <gazebo reference="head_mount">
         <material>Gazebo/Red</material>
     </gazebo>
@@ -27,5 +30,5 @@
         <material>Gazebo/Black</material>
     </gazebo>
-    <!-- Gazebo Plugins -->
+    <!-- General Gazebo Plugins -->
     <gazebo>
         <plugin name="gazebo_ros_control" filename="libgazebo_ros_control.so"></plugin>

File: urdf/studentbot/robot.xacro (robot description, xacro)
@@ -1,14 +1,174 @@
 <?xml version="1.0"?>
-<robot xmlns:xacro="http://www.ros.org/wiki/xacro" name="studentbot">
-    <xacro:include filename="$(find machine_vision_bonus)/urdf/studentbot/xacro/chasis.xacro"/>
-    <xacro:include filename="$(find machine_vision_bonus)/urdf/studentbot/xacro/wheels.xacro"/>
-    <xacro:include filename="$(find machine_vision_bonus)/urdf/studentbot/xacro/materials.xacro"/>
-    <xacro:include filename="$(find machine_vision_bonus)/urdf/studentbot/xacro/gazebo.xacro"/>
-    <!-- Robot Base Footprint -->
+<robot xmlns:xacro="http://www.ros.org/wiki/xacro" name="Differential Robot">
+    <xacro:property name="base_link_radius" value="0.0825" />
+    <xacro:property name="base_link_length" value="0.025" />
+    <xacro:property name="head_width" value="0.03" />
+    <xacro:property name="head_length" value="0.03" />
+    <xacro:property name="head_height" value="0.03" />
+    <xacro:property name="pi_over_2y" value="1.57075" />
+    <xacro:property name="pi_over_2z" value="1.57075" />
+    <xacro:property name="wheel_radius" value="0.035" />
+    <xacro:property name="wheel_length" value="0.008" />
+    <xacro:property name="passive_wheel_holder_radius" value="0.01" />
+    <xacro:property name="passive_wheel_holder_length" value="0.018" />
+    <xacro:property name="passive_wheel_holder_z_offset" value="-0.02" />
+    <xacro:macro name="wheel" params="prefix y_offset">
+        <link name="${prefix}_wheel">
+            <visual>
+                <origin xyz="0 0 0" rpy="0 ${pi_over_2y} ${pi_over_2z}" />
+                <geometry>
+                    <cylinder radius="${wheel_radius}" length="${wheel_length}" />
+                </geometry>
+                <material name="black"></material>
+            </visual>
+            <collision>
+                <origin xyz="0 0 0" rpy="0 ${pi_over_2y} ${pi_over_2z}" />
+                <geometry>
+                    <cylinder radius="${wheel_radius}" length="${wheel_length}" />
+                </geometry>
+            </collision>
+            <inertial>
+                <mass value="0.015"/>
+                <origin xyz="0 0 0" rpy="0 ${pi_over_2y} ${pi_over_2z}" />
+                <inertia ixx="0.00000467375" ixy="0.0" ixz="0.0" iyy="0.00000467375" iyz="0.0" izz="0.0000091875"/>
+            </inertial>
+        </link>
+        <joint name="base_to_${prefix}_wheel" type="continuous">
+            <axis xyz="0 1 0"/>
+            <origin xyz="0 ${y_offset} 0" rpy="0 0 0" />
+            <parent link="base_link"/>
+            <child link="${prefix}_wheel"/>
+        </joint>
+        <transmission name="base_to_${prefix}_wheel_trans">
+            <type>transmission_interface/SimpleTransmission</type>
+            <joint name="base_to_${prefix}_wheel">
+                <hardwareInterface>hardware_interface/VelocityJointInterface</hardwareInterface>
+            </joint>
+            <actuator name="${prefix}_wheel_motor">
+                <mechanicalReduction>1</mechanicalReduction>
+            </actuator>
+        </transmission>
+        <gazebo reference="${prefix}_wheel">
+            <mu1 value="200.0"/>
+            <mu2 value="100.0"/>
+            <kp value="10000000.0" />
+            <kd value="1.0" />
+            <material>Gazebo/Black</material>
+        </gazebo>
+    </xacro:macro>
+    <!-- Colors for Robot Parts -->
+    <material name="red">
+        <color rgba="1 0 0 1"/>
+    </material>
+    <material name="black">
+        <color rgba="0 0 0 1"/>
+    </material>
+    <material name="white">
+        <color rgba="1 1 1 1"/>
+    </material>
+    <material name="blue">
+        <color rgba="0 0 1 1"/>
+    </material>
+    <!-- Base Footprint Link -->
     <link name="base_footprint"></link>
-    <!-- Robot Chasis -->
-    <xacro:chasis />
-    <!-- Robot Wheels -->
-    <xacro:wheel prefix="left" offset="0.45" />
-    <xacro:wheel prefix="right" offset="-0.45" />
+    <joint name="base_footprint__base_link" type="fixed">
+        <origin xyz="0 0 0.035" rpy="0 0 0" />
+        <parent link="base_footprint"/>
+        <child link="base_link"/>
+    </joint>
+    <!-- Base Link -->
+    <link name="base_link">
+        <visual>
+            <geometry>
+                <cylinder radius="${base_link_radius}" length="${base_link_length}" />
+            </geometry>
+            <material name="red"></material>
+        </visual>
+        <collision>
+            <geometry>
+                <cylinder radius="${base_link_radius}" length="${base_link_length}" />
+            </geometry>
+        </collision>
+        <inertial>
+            <mass value="0.1"/>
+            <inertia ixx="0.0001753645833" ixy="0.0" ixz="0.0" iyy="0.0001753645833" iyz="0.0" izz="0.0003403125"/>
+        </inertial>
+    </link>
+    <!-- Head Link and Joint with Base Link -->
+    <joint name="base_to_head" type="fixed">
+        <origin xyz="0.065 0 0.025" rpy="0 0 0" />
+        <parent link="base_link"/>
+        <child link="head"/>
+    </joint>
+    <link name="head">
+        <visual>
+            <geometry>
+                <box size="${head_length} ${head_width} ${head_height}" />
+            </geometry>
+            <material name="blue"></material>
+        </visual>
+        <collision>
+            <geometry>
+                <box size="${head_length} ${head_width} ${head_height}" />
+            </geometry>
+        </collision>
+        <inertial>
+            <mass value="0.02"/>
+            <inertia ixx="0.000003" ixy="0.0" ixz="0.0" iyy="0.000003" iyz="0.0" izz="0.000003"/>
+        </inertial>
+    </link>
+    <!-- Left Wheel Link and Joint with Base Link -->
+    <xacro:wheel prefix="left" y_offset="0.0825" />
+    <!-- Right Wheel Link and Joint with Base Link -->
+    <xacro:wheel prefix="right" y_offset="-0.0825" />
+    <!-- Passive Wheel Holder Link and Joint with Base Link -->
+    <joint name="base_to_passive_wheel_holder" type="fixed">
+        <origin xyz="0.065 0 0" rpy="0 0 0" />
+        <parent link="base_link"/>
+        <child link="passive_wheel_holder"/>
+    </joint>
+    <link name="passive_wheel_holder">
+        <visual>
+            <origin xyz="0 0 ${passive_wheel_holder_z_offset}" />
+            <geometry>
+                <cylinder radius="${passive_wheel_holder_radius}" length="${passive_wheel_holder_length}" />
+            </geometry>
+            <material name="white"></material>
+        </visual>
+        <collision>
+            <origin xyz="0 0 ${passive_wheel_holder_z_offset}" />
+            <geometry>
+                <cylinder radius="${passive_wheel_holder_radius}" length="${passive_wheel_holder_length}" />
+            </geometry>
+        </collision>
+        <inertial>
+            <mass value="0.02"/>
+            <origin xyz="0 0 ${passive_wheel_holder_z_offset}" />
+            <inertia ixx="0.00000104" ixy="0.0" ixz="0.0" iyy="0.00000104" iyz="0.0" izz="0.000001"/>
+        </inertial>
+    </link>
+    <!-- Passive Wheel Link and Joint with Passive Wheel Holder Link -->
+    <joint name="base_to_passive_wheel" type="fixed">
+        <origin xyz="0 0 -0.025" rpy="0 0 0" />
+        <parent link="passive_wheel_holder"/>
+        <child link="passive_wheel"/>
+    </joint>
+    <link name="passive_wheel">
+        <visual>
+            <geometry>
+                <sphere radius="${passive_wheel_holder_radius}" />
+            </geometry>
+            <material name="white"></material>
+        </visual>
+        <collision>
+            <geometry>
+                <sphere radius="${passive_wheel_holder_radius}" />
+            </geometry>
+        </collision>
+        <inertial>
+            <mass value="0.02"/>
+            <inertia ixx="0.0000008" ixy="0.0" ixz="0.0" iyy="0.0000008" iyz="0.0" izz="0.0000008"/>
+        </inertial>
+    </link>
+    <xacro:include filename="gazebo.urdf" />
 </robot>
