Commit message: corrections based on supervisor feedback

File: urdf/ddrobot/xacro/chasis.xacro (robot description, xacro)
@@ -1,8 +1,13 @@
 <?xml version="1.0"?>
 <robot xmlns:xacro="http://www.ros.org/wiki/xacro">
-    <xacro:property name="head_mass" value="0.2" />
-    <xacro:property name="head_radius" value="0.15" />
+    <xacro:property name="head_mass" value="0.1" />
+    <xacro:property name="head_radius" value="0.25" />
     <xacro:property name="head_inertia_calc" value="${(2/5) * head_mass * (head_radius * head_radius)}" />
-    <xacro:property name="chasis_mass" value="0.1" />
+    <xacro:property name="head_mount_mass" value="0.1" />
+    <xacro:property name="head_mount_radius" value="0.1" />
+    <xacro:property name="head_mount_height" value="0.5" />
+    <xacro:property name="head_mount_inertia_calc" value="${(1/12) * head_mount_mass * ((3 * (head_mount_radius * head_mount_radius)) + (head_mount_height * head_mount_height))}" />
+    <xacro:property name="head_mount_inertia_calc_izz" value="${(1/2) * head_mount_mass * (head_mount_radius * head_mount_radius)}" />
+    <xacro:property name="chasis_mass" value="0.2" />
     <xacro:property name="chasis_width" value="0.8" />
     <xacro:property name="chasis_height" value="0.25" />
@@ -12,6 +17,6 @@
     <xacro:property name="chasis_inertia_calc_izz" value="${(1/12) * chasis_mass * ((chasis_width * chasis_width) + (chasis_length * chasis_length))}" />
     <xacro:macro name="chasis">
-        <!-- Robot Head Mount -->
-        <link name="head_mount">
+        <!-- Robot Head -->
+        <link name="head">
             <visual>
                 <origin xyz="0 0 0" rpy="0.0 0.0 0.0" />
@@ -32,6 +37,31 @@
             </inertial>
         </link>
+        <joint name="joint_head_mount__head" type="fixed">
+            <origin xyz="0 0 0.4" rpy="0.0 0.0 0.0" />
+            <parent link="head_mount"/>
+            <child link="head"/>
+        </joint>
+        <!-- Robot Head Mount -->
+        <link name="head_mount">
+            <visual>
+                <origin xyz="0 0 0" rpy="0 0 0"/>
+                <geometry>
+                    <cylinder radius="${head_mount_radius}" length="${head_mount_height}"/>
+                </geometry>
+                <material name="red"/>
+            </visual>
+            <collision>
+                <origin xyz="0 0 0" rpy="0 0 0"/>
+                <geometry>
+                    <cylinder radius="${head_mount_radius}" length="${head_mount_height}"/>
+                </geometry>
+            </collision>
+            <inertial>
+                <mass value="${head_mount_mass}"/>
+                <inertia ixx="${head_mount_inertia_calc}" ixy="0.0" ixz="0.0" iyy="${head_mount_inertia_calc}" iyz="0.0" izz="${head_mount_inertia_calc_izz}"/>
+            </inertial>
+        </link>
         <joint name="joint_chasis__head_mount" type="fixed">
-            <origin xyz="0.35 0 0.23" rpy="0.0 0.0 0.0" />
+            <origin xyz="0 0 0.23" rpy="0.0 0.0 0.0" />
             <parent link="chasis"/>
             <child link="head_mount"/>

File: urdf/ddrobot/xacro/gazebo.xacro (robot description, xacro)
@@ -1,7 +1,7 @@
 <?xml version="1.0"?>
 <robot xmlns:xacro="http://www.ros.org/wiki/xacro">
-    <xacro:macro name="robot_dynamics">
-        <mu1 value="200.0"/>
-        <mu2 value="100.0"/>
+    <xacro:macro name="robot_dynamics" params="mu1 mu2">
+        <mu1 value="${mu1}" />
+        <mu2 value="${mu2}" />
         <kp value="10000000.0" />
         <kd value="1.0" />
@@ -11,21 +11,24 @@
         <material>Gazebo/Red</material>
     </gazebo>
+    <gazebo reference="head">
+        <material>Gazebo/Red</material>
+    </gazebo>
     <gazebo reference="head_mount">
         <material>Gazebo/Red</material>
     </gazebo>
     <gazebo reference="right_front_wheel">
-        <xacro:robot_dynamics />
+        <xacro:robot_dynamics mu1="200" mu2="100" />
         <material>Gazebo/Black</material>
     </gazebo>
     <gazebo reference="right_back_wheel">
-        <xacro:robot_dynamics />
+        <xacro:robot_dynamics mu1="200" mu2="100" />
         <material>Gazebo/Black</material>
     </gazebo>
     <gazebo reference="left_front_wheel">
-        <xacro:robot_dynamics />
+        <xacro:robot_dynamics mu1="200" mu2="100" />
         <material>Gazebo/Black</material>
     </gazebo>
     <gazebo reference="left_back_wheel">
-        <xacro:robot_dynamics />
+        <xacro:robot_dynamics mu1="200" mu2="100" />
         <material>Gazebo/Black</material>
     </gazebo>
